File: dualusbserial.sch (KiCad schematic (older format))
At the start: 14 parts, among them IC1 CP2102, IC2 4N25, IC3 4N25, IC4 CP2102

Commit message: Initial PCB
Parts:
- removed USB2: MBUSB, symbol MBUSB
- added U1: MICRO-B_USB, ~, symbol MICRO-B_USB
Connections:
- net GND: no longer C4.1, C5.2, C6.1, IC3.2, IC4.3 (GND), R2.1
- net at IC4.4 (D+): now also U1.3 (D+)
- net at IC4.5 (D-): now also U1.2 (D-)
- net at C4.2, C6.2, IC4.7 (REGIN)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: now also U1.1 (VBUS)
- new net GNDA: C4.1, C5.2, C6.1, IC3.2, IC4.3 (GND), R2.1, U1.5 (GND)
Changed lines of the file:
@@
-$EndComp
-$Comp
-L MBUSB USB2
-U 1 1 5367E4FC
-P 7400 1600
-F 0 "USB2" H 7400 1200 60  0000 C CNN
-F 1 "MBUSB" H 7400 1950 60  0000 C CNN
-F 2 "" H 7400 1600 60  0000 C CNN
-F 3 "" H 7400 1600 60  0000 C CNN
-	1    7400 1600
-	0    1    -1   0
 $EndComp
 $Comp
@@
 $EndComp
 $Comp
-L GND #PWR6
-U 1 1 5367E508
-P 6700 1300
-F 0 "#PWR6" H 6700 1300 30  0001 C CNN
-F 1 "GND" H 6700 1230 30  0001 C CNN
-F 2 "" H 6700 1300 60  0000 C CNN
-F 3 "" H 6700 1300 60  0000 C CNN
-	1    6700 1300
-	-1   0    0    1
-$EndComp
-$Comp
 L C C6
 U 1 1 5367E50E
@@
 	1    6750 2550
 	-1   0    0    1
-$EndComp
-$Comp
-L GND #PWR5
-U 1 1 5367E514
-P 6600 2950
-F 0 "#PWR5" H 6600 2950 30  0001 C CNN
-F 1 "GND" H 6600 2880 30  0001 C CNN
-F 2 "" H 6600 2950 60  0000 C CNN
-F 3 "" H 6600 2950 60  0000 C CNN
-	1    6600 2950
-	1    0    0    -1
 $EndComp
 Wire Wire Line
@@
 Wire Wire Line
 	4800 2550 4550 2550
-$Comp
-L GND #PWR4
-U 1 1 5367E6F0
-P 4800 2700
-F 0 "#PWR4" H 4800 2700 30  0001 C CNN
-F 1 "GND" H 4800 2630 30  0001 C CNN
-F 2 "" H 4800 2700 60  0000 C CNN
-F 3 "" H 4800 2700 60  0000 C CNN
-	1    4800 2700
-	1    0    0    -1
-$EndComp
 Connection ~ 4800 2550
 Wire Wire Line
@@
 	0    -1   1    0
 $EndComp
+$Comp
+L MICRO-B_USB U1
+U 1 1 536907F8
+P 7300 1600
+F 0 "U1" H 7300 1300 50  0000 C CNN
+F 1 "MICRO-B_USB" H 7300 1900 50  0000 C CNN
+F 2 "~" H 7300 1600 60  0000 C CNN
+F 3 "~" H 7300 1600 60  0000 C CNN
+	1    7300 1600
+	-1   0    0    1
+$EndComp
+$Comp
+L GNDA #PWR?
+U 1 1 536920D0
+P 4800 2700
+F 0 "#PWR?" H 4800 2700 40  0001 C CNN
+F 1 "GNDA" H 4800 2630 40  0000 C CNN
+F 2 "" H 4800 2700 60  0000 C CNN
+F 3 "" H 4800 2700 60  0000 C CNN
+	1    4800 2700
+	1    0    0    -1
+$EndComp
+$Comp
+L GNDA #PWR?
+U 1 1 536920DF
+P 6700 1300
+F 0 "#PWR?" H 6700 1300 40  0001 C CNN
+F 1 "GNDA" H 6700 1230 40  0000 C CNN
+F 2 "" H 6700 1300 60  0000 C CNN
+F 3 "" H 6700 1300 60  0000 C CNN
+	1    6700 1300
+	-1   0    0    1
+$EndComp
+$Comp
+L GNDA #PWR?
+U 1 1 536920F8
+P 6600 2950
+F 0 "#PWR?" H 6600 2950 40  0001 C CNN
+F 1 "GNDA" H 6600 2880 40  0000 C CNN
+F 2 "" H 6600 2950 60  0000 C CNN
+F 3 "" H 6600 2950 60  0000 C CNN
+	1    6600 2950
+	1    0    0    -1
+$EndComp
 $EndSCHEMATC
